Commit message: revise foosball table urdf

File: foosball.urdf (robot description, URDF)
Before this commit: robot foosball_table_tuned_v2, 41 links, 40 joints
Links:
- added link p1_2, mass 0.1; collision cylinder length=0.13 radius=0.015; visual cylinder length=0.13 radius=0.015
- added link p1_3, mass 0.1; collision cylinder length=0.13 radius=0.015; visual cylinder length=0.13 radius=0.015
- added link p8_2, mass 0.1; collision cylinder length=0.13 radius=0.015; visual cylinder length=0.13 radius=0.015
- added link p8_3, mass 0.1; collision cylinder length=0.13 radius=0.015; visual cylinder length=0.13 radius=0.015
- link base_link: geometry collision box size=0.05 0.24 0.15; collision box size=0.05 0.24 0.15
Joints:
- added joint p1_2_j: type fixed, parent rod_1_link, child p1_2, origin xyz=0 0.20 0
- added joint p1_3_j: type fixed, parent rod_1_link, child p1_3, origin xyz=0 -0.20 0
- added joint p8_2_j: type fixed, parent rod_8_link, child p8_2, origin xyz=0 0.20 0
- added joint p8_3_j: type fixed, parent rod_8_link, child p8_3, origin xyz=0 -0.20 0
- joint goal_sensor_A_joint: origin xyz=-0.60 0 0.05 -> xyz=-0.75 0 0.05
- joint goal_sensor_B_joint: origin xyz=0.60 0 0.05 -> xyz=0.75 0 0.05
- joint p2_1_j: origin xyz=0 0.22 0 -> xyz=0 0.14 0
- joint p2_2_j: origin xyz=0 -0.22 0 -> xyz=0 -0.14 0
- joint p7_1_j: origin xyz=0 0.22 0 -> xyz=0 0.14 0
- joint p7_2_j: origin xyz=0 -0.22 0 -> xyz=0 -0.14 0
- joint rod_2_slide: limit lower=-0.10 upper=0.10 effort=100 velocity=10 -> lower=-0.18 upper=0.18 effort=100 velocity=10
- joint rod_7_slide: limit lower=-0.10 upper=0.10 effort=100 velocity=10 -> lower=-0.18 upper=0.18 effort=100 velocity=10

Commit message: change urdf file and reward function again

File: foosball.urdf (robot description, URDF)
Before this commit: robot foosball_table_tuned_v2, 45 links, 44 joints
Joints:
- joint rod_1_slide: origin xyz=-0.55 0 0.15 -> xyz=-0.625 0 0.15
- joint rod_2_slide: origin xyz=-0.40 0 0.15 -> xyz=-0.45 0 0.15
- joint rod_3_slide: origin xyz=-0.25 0 0.15 -> xyz=-0.275 0 0.15
- joint rod_6_slide: origin xyz=0.25 0 0.15 -> xyz=0.275 0 0.15
- joint rod_7_slide: origin xyz=0.40 0 0.15 -> xyz=0.45 0 0.15
- joint rod_8_slide: origin xyz=0.55 0 0.15 -> xyz=0.625 0 0.15

Commit message: change structure

File: foosball.urdf (robot description, URDF)
Before this commit: robot foosball_table_tuned_v2, 45 links, 44 joints
Joints:
- joint goal_sensor_A_joint: origin xyz=-0.75 0 0.05 -> xyz=-0.70 0 0.05
- joint goal_sensor_B_joint: origin xyz=0.75 0 0.05 -> xyz=0.70 0 0.05

Commit message: change table

File: foosball.urdf (robot description, URDF)
Before this commit: robot foosball_table_tuned_v2, 45 links, 44 joints
Links:
- link base_link: geometry collision box size=0.075 0.24 0.15; collision box size=0.075 0.24 0.15
Joints:
- joint goal_sensor_A_joint: origin xyz=-0.70 0 0.05 -> xyz=-0.73 0 0.05
- joint goal_sensor_B_joint: origin xyz=0.70 0 0.05 -> xyz=0.73 0 0.05

Commit message: i hate gemini

File: foosball.urdf (robot description, URDF)
Before this commit: robot foosball_table_tuned_v2, 45 links, 44 joints
Links:
- link rod_1_link: mass 0.5 -> 0.01
- link rod_2_link: mass 0.5 -> 0.01
- link rod_3_link: mass 0.5 -> 0.01
- link rod_4_link: mass 0.5 -> 0.01
- link rod_5_link: mass 0.5 -> 0.01
- link rod_6_link: mass 0.5 -> 0.01
- link rod_7_link: mass 0.5 -> 0.01
- link rod_8_link: mass 0.5 -> 0.01

Commit message: pray

File: foosball.urdf (robot description, URDF)
Before this commit: robot foosball_table_tuned_v2, 45 links, 44 joints
Links:
- link p1_1: geometry collision box size=0.02 0.03 0.13; visual box size=0.02 0.03 0.13
- link p1_2: geometry collision box size=0.02 0.03 0.13; visual box size=0.02 0.03 0.13
- link p1_3: geometry collision box size=0.02 0.03 0.13; visual box size=0.02 0.03 0.13
- link p2_1: geometry collision box size=0.02 0.03 0.13; visual box size=0.02 0.03 0.13
- link p2_2: geometry collision box size=0.02 0.03 0.13; visual box size=0.02 0.03 0.13
- link p3_1: geometry collision box size=0.02 0.03 0.13; visual box size=0.02 0.03 0.13
- link p3_2: geometry collision box size=0.02 0.03 0.13; visual box size=0.02 0.03 0.13
- link p3_3: geometry collision box size=0.02 0.03 0.13; visual box size=0.02 0.03 0.13
- link p4_1: geometry collision box size=0.02 0.03 0.13; visual box size=0.02 0.03 0.13
- link p4_2: geometry collision box size=0.02 0.03 0.13; visual box size=0.02 0.03 0.13
- link p4_3: geometry collision box size=0.02 0.03 0.13; visual box size=0.02 0.03 0.13
- link p4_4: geometry collision box size=0.02 0.03 0.13; visual box size=0.02 0.03 0.13
- link p4_5: geometry collision box size=0.02 0.03 0.13; visual box size=0.02 0.03 0.13
- link p5_1: geometry collision box size=0.02 0.03 0.13; visual box size=0.02 0.03 0.13
- link p5_2: geometry collision box size=0.02 0.03 0.13; visual box size=0.02 0.03 0.13
- link p5_3: geometry collision box size=0.02 0.03 0.13; visual box size=0.02 0.03 0.13
- link p5_4: geometry collision box size=0.02 0.03 0.13; visual box size=0.02 0.03 0.13
- link p5_5: geometry collision box size=0.02 0.03 0.13; visual box size=0.02 0.03 0.13
- link p6_1: geometry collision box size=0.02 0.03 0.13; visual box size=0.02 0.03 0.13
- link p6_2: geometry collision box size=0.02 0.03 0.13; visual box size=0.02 0.03 0.13
- link p6_3: geometry collision box size=0.02 0.03 0.13; visual box size=0.02 0.03 0.13
- link p7_1: geometry collision box size=0.02 0.03 0.13; visual box size=0.02 0.03 0.13
- link p7_2: geometry collision box size=0.02 0.03 0.13; visual box size=0.02 0.03 0.13
- link p8_1: geometry collision box size=0.02 0.03 0.13; visual box size=0.02 0.03 0.13
- link p8_2: geometry collision box size=0.02 0.03 0.13; visual box size=0.02 0.03 0.13
- link p8_3: geometry collision box size=0.02 0.03 0.13; visual box size=0.02 0.03 0.13
